Commit message: tf renewed

File: robot_core/urdf/minibase_urdf.xacro (robot description, xacro)
@@ -1,23 +1,7 @@
 <?xml version="1.0"?>
 <robot name="robot" xmlns:xacro="http://ros.org/wiki/xacro">
-  <xacro:arg name="LIDAR_MODEL" default="pacecat"/> <!-- pacecat, pacecat_cr, rplidar -->
-  <xacro:arg name="base_color" default="0.45 0.48 0.50 1.0"/>
-  <xacro:arg name="x_offset" default="0.15"/>
-  <xacro:arg name="z_offset" default="0.43"/>
-  <xacro:arg name="pitch_angle" default="-0.6"/>
-  <xacro:property name="LIDAR_MODEL" value="$(arg LIDAR_MODEL)"/>
-  <xacro:property name="lidar_frame" value="scan_central_link"/>
-  <!-- Medidas exactas de posicion del lidar en el robot real con respecto al -->
-  <!-- marco base_link (punto medio del eje de las ruedas con 'wheelRadius' sobre Z) -->
-  <xacro:property name="lidar_offset_x" value="0.24"/>
-  <xacro:property name="lidar_offset_y" value="0.0"/>
-  <!-- Medidas que pueden no ser exactas, solo para visualizar al robot -->
-  <xacro:property name="lidar_offset_z" value="0.33"/>
-  <xacro:property name="wheelRadius" value="0.065"/>
-  <xacro:property name="wheelSeparation" value="0.36"/>
-  <xacro:property name="wheelThickness" value="0.09"/>
-  <xacro:property name="baseLength" value="0.45"/>
-  <xacro:property name="baseWidth" value="${wheelSeparation-0.06}"/>
-  <xacro:property name="baseHeight" value="${wheelRadius-0.02}"/>
+  <!-- ========================================================== -->
+  <!--                 CONSTANTES Y MACROS                        -->
+  <!-- ========================================================== -->
   <xacro:property name="PI" value="3.14159265"/>
   <xacro:macro name="box_inertial" params="mass x y z">
@@ -54,13 +38,19 @@
     </inertial>
   </xacro:macro>
+  <!-- ========================================================== -->
+  <!--                       CHASIS                               -->
+  <!-- ========================================================== -->
+  <!-- Argumentos y Propiedades -->
+  <xacro:arg name="base_color" default="0.45 0.48 0.50 1.0"/>
+  <xacro:property name="wheelSeparation" value="0.35"/>
+  <xacro:property name="wheelRadius" value="0.06"/>
+  <xacro:property name="baseLength" value="0.55"/>
+  <xacro:property name="baseWidth" value="${wheelSeparation-0.06}"/>
+  <xacro:property name="baseHeight" value="${wheelRadius-0.02}"/>
+  <!-- Materiales -->
   <material name="base_gray">
     <color rgba="$(arg base_color)"/>
   </material>
-  <material name="wheel_black">
-    <color rgba="0.02 0.02 0.02 1.0"/>
-  </material>
-  <material name="lidar_black">
-    <color rgba="0.0 0.0 0.0 1.0"/>
-  </material>
+  <!-- Enlaces y Articulaciones -->
   <link name="base_footprint">
     <xacro:dummy_inertial/>
@@ -87,5 +77,15 @@
     <xacro:box_inertial mass="8.0" x="${baseLength}" y="${baseWidth}" z="${baseHeight}"/>
   </link>
-  <!-- Wheels definition (fixed, not continuous) -->
+  <!-- ========================================================== -->
+  <!--                       LLANTAS                              -->
+  <!-- ========================================================== -->
+  <!-- Propiedades -->
+  <xacro:property name="wheelThickness" value="0.09"/>
+  <!-- Materiales -->
+  <material name="wheel_black">
+    <color rgba="0.02 0.02 0.02 1.0"/>
+  </material>
+  <!-- Enlaces y Articulaciones -->
+  <!-- Rueda Izquierda -->
   <joint name="wheel_left_joint" type="fixed">
     <parent link="base_link"/>
@@ -110,4 +110,5 @@
     <xacro:cylinder_inertial mass="0.8" radius="${wheelRadius}" length="${wheelThickness}"/>
   </link>
+  <!-- Rueda Derecha -->
   <joint name="wheel_right_joint" type="fixed">
     <parent link="base_link"/>
@@ -132,23 +133,60 @@
     <xacro:cylinder_inertial mass="0.8" radius="${wheelRadius}" length="${wheelThickness}"/>
   </link>
-  <!-- SENSORS definition -->
-  <!-- IMU -->
+  <!-- ========================================================== -->
+  <!--                       SENSORES                             -->
+  <!-- ========================================================== -->
+  <!-- ======================= IMU ======================= -->
+  <xacro:arg name="imu_offset_x" default="0.065"/>
+  <xacro:arg name="imu_offset_y" default="0.0"/>
+  <xacro:arg name="imu_offset_z" default="0.24"/>
+  <xacro:arg name="imu_offset_roll" default="0.0"/>
+  <xacro:arg name="imu_offset_pitch" default="0.0"/>
+  <xacro:arg name="imu_offset_yaw" default="0.0"/>
   <joint name="imu_joint" type="fixed">
     <parent link="base_link"/>
     <child link="imu_link"/>
-    <origin xyz="0 0 0" rpy="0 0 0"/>
-  </joint>
+    <origin xyz="$(arg imu_offset_x) $(arg imu_offset_y) $(arg imu_offset_z)" rpy="$(arg imu_offset_roll) $(arg imu_offset_pitch) $(arg imu_offset_yaw)"/>
+  </joint>
+  <material name="imu_blue">
+    <color rgba="0.2 0.3 0.8 1.0"/>
+  </material>
   <link name="imu_link">
-    <xacro:dummy_inertial/>
-  </link>
-  <!-- LIDAR -->
+    <visual>
+      <origin xyz="0 0 0" rpy="0 0 0"/>
+      <geometry>
+        <box size="0.06 0.06 0.06"/>
+      </geometry>
+      <material name="imu_blue"/>
+    </visual>
+    <collision>
+      <origin xyz="0 0 0" rpy="0 0 0"/>
+      <geometry>
+        <box size="0.06 0.06 0.06"/>
+      </geometry>
+    </collision>
+    <xacro:box_inertial mass="0.1" x="0.06" y="0.06" z="0.06"/>
+  </link>
+  <!-- ====================== LIDAR ====================== -->
+  <xacro:arg name="LIDAR_MODEL" default="pacecat"/> <!-- pacecat, pacecat_cr, rplidar -->
+  <xacro:arg name="lidar_offset_x" default="0.2125"/>
+  <xacro:arg name="lidar_offset_y" default="0.0"/>
+  <xacro:arg name="lidar_offset_z" default="0.24"/>
+  <xacro:arg name="lidar_offset_roll" default="0.0"/>
+  <xacro:arg name="lidar_offset_pitch" default="0.0"/>
+  <xacro:arg name="lidar_offset_yaw" default="0.0"/>
+  <xacro:property name="LIDAR_MODEL" value="$(arg LIDAR_MODEL)"/>
+  <xacro:property name="lidar_frame" value="scan_central_link"/>
+  <xacro:property name="lidar_yaw_val" value="$(arg lidar_offset_yaw)"/>
+  <material name="lidar_black">
+    <color rgba="0.0 0.0 0.0 1.0"/>
+  </material>
   <joint name="lidar_joint" type="fixed">
     <parent link="base_link"/>
     <child link="${lidar_frame}"/>
     <xacro:if value="${LIDAR_MODEL == 'pacecat'}" >
-      <origin xyz="${lidar_offset_x} ${lidar_offset_y} ${lidar_offset_z}" rpy="0 0 0"/>
+      <origin xyz="$(arg lidar_offset_x) $(arg lidar_offset_y) $(arg lidar_offset_z)" rpy="0 0 0"/>
     </xacro:if>
     <xacro:if value="${LIDAR_MODEL == 'rplidar'}" >
-      <origin xyz="${lidar_offset_x} ${lidar_offset_y} ${lidar_offset_z}" rpy="0 0 ${PI}"/>
+      <origin xyz="$(arg lidar_offset_x) $(arg lidar_offset_y) $(arg lidar_offset_z)" rpy="0 0 ${PI}"/>
     </xacro:if>
   </joint>
@@ -157,5 +195,5 @@
       <origin xyz="0 0 0" rpy="0 0 0"/>
       <geometry>
-        <cylinder length="0.06" radius="0.05"/>
+        <cylinder length="0.06" radius="0.0275"/>
       </geometry>
       <material name="lidar_black"/>
@@ -164,27 +202,69 @@
       <origin xyz="0 0 0" rpy="0 0 0"/>
       <geometry>
-        <cylinder length="0.06" radius="0.05"/>
-      </geometry>
-    </collision>
-    <xacro:cylinder_inertial mass="0.2" radius="0.05" length="0.06"/>
-  </link>
-  <!-- CLOUD CAMERA -->
-  <!-- Realsense -->
-  <joint name="cloud_joint" type="fixed">
-    <parent link="base_link"/>
-    <child link="camera_link"/>
-    <origin xyz="$(arg x_offset) 0 $(arg z_offset)" rpy="0 $(arg pitch_angle) 0"/>
-  </joint>
-  <link name="camera_link">
-    <xacro:dummy_inertial/>
-  </link>
-  <!-- Frontal Camera -->
-  <joint name="frontal_cam_joint" type="fixed">
-    <parent link="base_footprint"/>
-    <child link="frontal_camera_link"/>
-    <origin xyz="0.1 0.0 1.25" rpy="0 0 0"/>
-  </joint>
-  <link name="frontal_camera_link">
-    <xacro:dummy_inertial/>
-  </link>
+        <cylinder length="0.055" radius="0.055"/>
+      </geometry>
+    </collision>
+    <xacro:cylinder_inertial mass="0.2" radius="0.055" length="0.055"/>
+  </link>
+  <!-- ===================== KINECT ====================== -->
+  <xacro:arg name="kinect_offset_x" default="0.115"/>
+  <xacro:arg name="kinect_offset_y" default="0.0"/>
+  <xacro:arg name="kinect_offset_z" default="0.39"/>
+  <xacro:arg name="kinect_offset_roll" default="0.0"/>
+  <xacro:arg name="kinect_offset_pitch" default="0.0"/>
+  <xacro:arg name="kinect_offset_yaw" default="0.0"/>
+  <joint name="kinect_joint" type="fixed">
+    <parent link="base_link"/>
+    <child link="camera_base"/>
+    <origin xyz="$(arg kinect_offset_x) $(arg kinect_offset_y) $(arg kinect_offset_z)" rpy="$(arg kinect_offset_roll) $(arg kinect_offset_pitch) $(arg kinect_offset_yaw)"/>
+  </joint>
+  <material name="kinect_black">
+    <color rgba="0. 0. 0. 1" />
+  </material>
+  <material name="kinect_dark_grey">
+    <color rgba="0.1 0.1 0.1 1" />
+  </material>
+  <material name="kinect_grey">
+    <color rgba="0.6 0.6 0.6 1" />
+  </material>
+  <material name="kinect_white">
+    <color rgba="0.9 0.9 0.9 1" />
+  </material>
+  <link name="camera_body">
+    <visual>
+      <origin xyz="0. 0. 0." />
+      <geometry>
+        <box size="0.0994 0.0996 0.023" />
+      </geometry>
+      <material name="kinect_white" />
+    </visual>
+  </link>
+  <link name="camera_base">
+    <visual>
+      <origin xyz="-0.013 0. 0." />
+      <geometry>
+        <box size="0.026 0.103 0.039" />
+      </geometry>
+      <material name="kinect_grey" />
+    </visual>
+  </link>
+  <link name="camera_visor">
+    <visual>
+      <origin xyz="-0.0128 0. 0." />
+      <geometry>
+        <box size="0.026 0.101 0.037" />
+      </geometry>
+      <material name="kinect_black" />
+    </visual>
+  </link>
+  <joint name="camera_base_to_body" type="fixed">
+    <parent link="camera_base" />
+    <child link="camera_body" />
+    <origin xyz="-0.0757 0. 0.008" rpy="0. 0. 0." />
+  </joint>
+  <joint name="camera_base_to_visor" type="fixed">
+    <parent link="camera_base" />
+    <child link="camera_visor" />
+    <origin xyz="0. 0. 0." rpy="0. 0. 0." />
+  </joint>
 </robot>

Commit message: changes in URDF

File: robot_core/urdf/minibase_urdf.xacro (robot description, xacro)
@@ -44,5 +44,5 @@
   <xacro:arg name="base_color" default="0.45 0.48 0.50 1.0"/>
   <xacro:property name="wheelSeparation" value="0.35"/>
-  <xacro:property name="wheelRadius" value="0.06"/>
+  <xacro:property name="wheelRadius" value="0.1"/>
   <xacro:property name="baseLength" value="0.55"/>
   <xacro:property name="baseWidth" value="${wheelSeparation-0.06}"/>

Commit message: Add rover simulation package and configuration for Gazebo Harmonic simulation
- Created `rover_simulation` package with CMakeLists.txt and package.xml.
- Added configuration files for EKF and ros_gz_bridge.
- Implemented launch file for simulation bringup, including optional components like RTAB-Map and path planning.
- Updated voice_bt behavior to support dynamic topic configuration for RTAB-Map in both hardware and simulation environments.
- Added RViz configuration for visualization of the simulation.
- Included necessary dependencies in package.xml for proper functionality.

File: robot_core/urdf/minibase_urdf.xacro (robot description, xacro)
@@ -38,4 +38,17 @@
     </inertial>
   </xacro:macro>
+  <xacro:macro name="sphere_inertial" params="mass radius">
+    <inertial>
+      <origin xyz="0 0 0" rpy="0 0 0"/>
+      <mass value="${mass}"/>
+      <inertia
+        ixx="${2.0 * mass * radius*radius / 5.0}"
+        ixy="0.0"
+        ixz="0.0"
+        iyy="${2.0 * mass * radius*radius / 5.0}"
+        iyz="0.0"
+        izz="${2.0 * mass * radius*radius / 5.0}"/>
+    </inertial>
+  </xacro:macro>
   <!-- ========================================================== -->
   <!--                       CHASIS                               -->
@@ -43,4 +56,6 @@
   <!-- Argumentos y Propiedades -->
   <xacro:arg name="base_color" default="0.45 0.48 0.50 1.0"/>
+  <xacro:arg name="sim" default="false"/>
+  <xacro:property name="sim_mode" value="$(arg sim)"/>
   <xacro:property name="wheelSeparation" value="0.35"/>
   <xacro:property name="wheelRadius" value="0.1"/>
@@ -88,5 +103,5 @@
   <!-- Enlaces y Articulaciones -->
   <!-- Rueda Izquierda -->
-  <joint name="wheel_left_joint" type="fixed">
+  <joint name="wheel_left_joint" type="${'continuous' if sim_mode else 'fixed'}">
     <parent link="base_link"/>
     <child link="wheel_left_link"/>
@@ -111,5 +126,5 @@
   </link>
   <!-- Rueda Derecha -->
-  <joint name="wheel_right_joint" type="fixed">
+  <joint name="wheel_right_joint" type="${'continuous' if sim_mode else 'fixed'}">
     <parent link="base_link"/>
     <child link="wheel_right_link"/>
@@ -133,4 +148,42 @@
     <xacro:cylinder_inertial mass="0.8" radius="${wheelRadius}" length="${wheelThickness}"/>
   </link>
+  <!-- ========================================================== -->
+  <!--                    SWIVEL CASTERS                          -->
+  <!-- ========================================================== -->
+  <!-- Ball casters (sphere r=0.03 m) placed under the chassis    -->
+  <!-- front and rear to prevent tipping. Zero friction is set    -->
+  <!-- in the sim overlay so they slide freely like real swivels. -->
+  <xacro:property name="casterRadius" value="0.03"/>
+  <!-- z offset puts the sphere centre at exactly ground level    -->
+  <!-- base_link is wheelRadius above ground, so:                 -->
+  <!--   z = casterRadius - wheelRadius = 0.03 - 0.10 = -0.07    -->
+  <xacro:property name="casterZ" value="${casterRadius - wheelRadius}"/>
+  <!-- x offset: inset ~5 cm from each end of the chassis         -->
+  <xacro:property name="casterX" value="${baseLength/2 - 0.05}"/>
+  <xacro:macro name="swivel_caster" params="prefix x_pos">
+    <joint name="caster_${prefix}_joint" type="fixed">
+      <parent link="base_link"/>
+      <child link="caster_${prefix}_link"/>
+      <origin xyz="${x_pos} 0 ${casterZ}" rpy="0 0 0"/>
+    </joint>
+    <link name="caster_${prefix}_link">
+      <visual>
+        <origin xyz="0 0 0" rpy="0 0 0"/>
+        <geometry>
+          <sphere radius="${casterRadius}"/>
+        </geometry>
+        <material name="wheel_black"/>
+      </visual>
+      <collision>
+        <origin xyz="0 0 0" rpy="0 0 0"/>
+        <geometry>
+          <sphere radius="${casterRadius}"/>
+        </geometry>
+      </collision>
+      <xacro:sphere_inertial mass="0.1" radius="${casterRadius}"/>
+    </link>
+  </xacro:macro>
+  <xacro:swivel_caster prefix="front" x_pos="${casterX}"/>
+  <xacro:swivel_caster prefix="rear"  x_pos="${-casterX}"/>
   <!-- ========================================================== -->
   <!--                       SENSORES                             -->
@@ -268,3 +321,24 @@
     <origin xyz="0. 0. 0." rpy="0. 0. 0." />
   </joint>
+  <!-- ===================== SIM-ONLY FRAMES ===================== -->
+  <!-- These frames are required in simulation for RTAB-Map and   -->
+  <!-- pointcloud_roi_node which reference depth_camera_link.     -->
+  <xacro:if value="${sim_mode}">
+    <link name="depth_camera_link">
+      <xacro:dummy_inertial/>
+    </link>
+    <joint name="camera_base_to_depth_link" type="fixed">
+      <parent link="camera_base"/>
+      <child link="depth_camera_link"/>
+      <origin xyz="0 0 0" rpy="0 0 0"/>
+    </joint>
+    <link name="depth_camera_optical_frame">
+      <xacro:dummy_inertial/>
+    </link>
+    <joint name="camera_base_to_optical" type="fixed">
+      <parent link="camera_base"/>
+      <child link="depth_camera_optical_frame"/>
+      <origin xyz="0 0 0" rpy="0 0 0"/>
+    </joint>
+  </xacro:if>
 </robot>

Commit message: fix: adjust camera joint orientation and update point cloud handling in simulation

File: robot_core/urdf/minibase_urdf.xacro (robot description, xacro)
@@ -339,5 +339,5 @@
       <parent link="camera_base"/>
       <child link="depth_camera_optical_frame"/>
-      <origin xyz="0 0 0" rpy="0 0 0"/>
+      <origin xyz="0 0 0" rpy="${-PI/2} 0 ${-PI/2}"/>
     </joint>
   </xacro:if>

Commit message: refactor 706 robot added

File: robot_core/urdf/minibase_urdf.xacro (robot description, xacro)
@@ -57,6 +57,7 @@
   <xacro:arg name="base_color" default="0.45 0.48 0.50 1.0"/>
   <xacro:arg name="sim" default="false"/>
+  <xacro:arg name="wheel_separation" default="0.315"/>
   <xacro:property name="sim_mode" value="$(arg sim)"/>
-  <xacro:property name="wheelSeparation" value="0.35"/>
+  <xacro:property name="wheelSeparation" value="$(arg wheel_separation)"/>
   <xacro:property name="wheelRadius" value="0.1"/>
   <xacro:property name="baseLength" value="0.55"/>
@@ -263,5 +264,5 @@
   <xacro:arg name="kinect_offset_x" default="0.115"/>
   <xacro:arg name="kinect_offset_y" default="0.0"/>
-  <xacro:arg name="kinect_offset_z" default="0.39"/>
+  <xacro:arg name="kinect_offset_z" default="0.30"/>
   <xacro:arg name="kinect_offset_roll" default="0.0"/>
   <xacro:arg name="kinect_offset_pitch" default="0.0"/>
